File: hardware/pokey-synth.brd (EAGLE design)
At the start: 120.7 x 69.8 mm, 51 parts, among them IC1 MEGA8-P, IC2 POKEYDIP40, IC3 POKEYDIP40, IC4 6N138

Commit message: updates
Parts:
- moved C9 3.18 mm to (118.7, 57.8), turned to 0 degrees
- moved C10 2.01 mm to (118.7, 39.4), turned to 0 degrees
- moved C12 1.27 mm to (121.9, 50.8)
- moved C13 1.27 mm to (121.9, 45.7)
- moved U$8 0.76 mm to (119.4, 94.7)
Connections:
- net GND: now also R4.1
Routing:
- net VCC: track 289.0 -> 282.4 mm, vias 1 -> 2
- net N$28: track 49.3 -> 55.8 mm
- net N$24: track 30.8 -> 31.8 mm
- net N$20: track 7.91 -> 8.97 mm
- net N$18: track 15.8 -> 15.1 mm
Other:
- outline, holes or cut-outs redrawn
- board text added: "BATT"
- board text added: "POKEY synth rev 1"
- board text added: "hotchk155"
