File: hardware/pokey-synth.brd (EAGLE design)
At the start: 120.7 x 69.8 mm, 51 parts, among them IC1 MEGA8-P, IC2 POKEYDIP40, IC3 POKEYDIP40, IC4 6N138

Commit message: pcb ready
Parts:
- moved C7 0.76 mm to (87.6, 56.6)
Routing:
- net VCC: track 282.4 -> 283.1 mm

Commit message: more stuff
Parts:
- R6, R7: value (none) -> 470
Connections:
- removed net N$6: OUT_A/MIX.RING, OUT_A/MIX.RING_NC, OUT_B.TIP_NC
- net N$5: now also OUT_B.TIP_NC
Routing:
- net N$6: track 24.7 -> 0.00 mm
- net N$5: track 17.2 -> 37.4 mm
Changed lines of the file:
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@@
 <attribute name="VALUE" x="35.306" y="75.4888" size="1.27" layer="27" ratio="10" rot="R180"/>
 </element>
-<element name="R7" library="rcl" package="0207/7" value="" x="43.815" y="76.2" smashed="yes" rot="R270">
+<element name="R7" library="rcl" package="0207/7" value="470" x="43.815" y="76.2" smashed="yes" rot="R270">
 <attribute name="NAME" x="43.307" y="77.47" size="1.27" layer="25" ratio="10" rot="R270"/>
 <attribute name="VALUE" x="43.2562" y="78.486" size="1.27" layer="27" ratio="10" rot="R270"/>
@@
 <attribute name="NAME" x="14.859" y="62.484" size="1.27" layer="25" ratio="10"/>
 </element>
-<element name="R6" library="rcl" package="0207/7" value="" x="40.64" y="76.2" smashed="yes" rot="R270">
+<element name="R6" library="rcl" package="0207/7" value="470" x="40.64" y="76.2" smashed="yes" rot="R270">
 <attribute name="NAME" x="40.132" y="77.47" size="1.27" layer="25" ratio="10" rot="R270"/>
 <attribute name="VALUE" x="40.0812" y="78.486" size="1.27" layer="27" ratio="10" rot="R270"/>
@@
 <wire x1="87.63" y1="82.55" x2="84.455" y2="79.375" width="0.4064" layer="1"/>
 <wire x1="81.28" y1="79.375" x2="84.455" y2="79.375" width="0.4064" layer="1"/>
-</signal>
-<signal name="N$6">
-<contactref element="OUT_A/MIX" pad="RING"/>
-<contactref element="OUT_A/MIX" pad="RING_NC"/>
 <contactref element="OUT_B" pad="TIP_NC"/>
-<wire x1="95.25" y1="89.535" x2="97.79" y2="89.535" width="0.4064" layer="16"/>
 <wire x1="94.615" y1="92.075" x2="78.105" y2="92.075" width="0.4064" layer="16"/>
 <wire x1="78.105" y1="92.075" x2="77.47" y2="91.44" width="0.4064" layer="16"/>
 <wire x1="77.47" y1="91.44" x2="77.47" y2="89.535" width="0.4064" layer="16"/>
-<wire x1="95.25" y1="89.535" x2="95.25" y2="91.44" width="0.4064" layer="16"/>
 <wire x1="95.25" y1="91.44" x2="94.615" y2="92.075" width="0.4064" layer="16"/>
+<wire x1="90.17" y1="89.535" x2="94.615" y2="92.075" width="0" layer="19" extent="16-16"/>
 </signal>
 <signal name="N$7">

Commit message: add jumper
Parts:
- added JP3: (no value), pinhead:1X03
- moved SERIAL 23.6 mm to (10.2, 43.2)
- moved OUT_A/MIX 12.7 mm to (80.0, 90.8)
- moved OUT_B 12.7 mm to (92.7, 90.8)
Connections:
- net CS1: now also JP3.1
- net GND: now also JP3.2
Routing:
- net N$21: track 2.54 -> 33.8 mm
- net TXD: track 5.08 -> 34.5 mm
- net RXD: track 31.4 -> 47.8 mm
- net VCC: track 283.1 -> 297.1 mm
- net N$5: track 37.4 -> 33.6 mm
- net GND: track 16.1 -> 12.5 mm
- net N$10: track 11.1 -> 12.6 mm
- net CS1: track 42.4 -> 43.1 mm, vias 1 -> 0
Other:
- board text added: "1"
- board text added: "DUAL"
- board text added: "POKEY"
- board text added: "POKEY synth"
- board text added: "SINGLE"
- board text added: "rev 2"
- board text removed: "POKEY synth rev 1"
