File: hardware/pokey-synth.brd (EAGLE design)
At the start: 120.7 x 69.8 mm, 52 parts, among them IC1 MEGA8-P, IC2 POKEYDIP40, IC3 POKEYDIP40, IC4 6N138

Commit message: updates
Parts:
- moved IC1 1.27 mm to (33.0, 55.9)
- moved R4 1.27 mm to (20.3, 40.0)
- moved X1 1.27 mm to (24.1, 49.5)
- moved LED1 1.27 mm to (110.5, 34.3)
- moved LED2 1.27 mm to (100.3, 34.3)
- moved LED3 1.27 mm to (30.5, 34.3)
- moved MODE 1.27 mm to (20.3, 34.3)
- moved R5 1.27 mm to (33.0, 76.2)
Routing:
- net GND: track 12.5 -> 9.94 mm
- net N$26: track 101.4 -> 103.7 mm
- net DB3: track 41.3 -> 39.2 mm, vias 0 -> 1
- net N$2: track 11.7 -> 13.8 mm
- net DB2: track 56.2 -> 54.9 mm
- net AD3: track 66.3 -> 65.1 mm
- net DB0: track 58.0 -> 56.7 mm
- net N$27: track 4.71 -> 3.44 mm
- net N$25: track 7.51 -> 6.24 mm
- net DB1: track 58.0 -> 56.7 mm
- net CS0: track 49.3 -> 48.0 mm
- net N$28: track 55.8 -> 57.1 mm
- net RXD: track 47.8 -> 46.8 mm
- net VCC: track 297.1 -> 297.9 mm
- net N$30: track 9.99 -> 10.7 mm
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