File: hardware/pokey-synth.sch (EAGLE design)
At the start: 51 parts, among them IC1 MEGA8-P, IC2 POKEYDIP40, IC3 POKEYDIP40, IC4 6N138

Commit message: updates
Connections:
- net GND: now also R4.1
Other:
- moved on the sheet: C3, U$8
Changed lines of the file:
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@@
 <instance part="R3" gate="G$1" x="88.9" y="-12.7"/>
 <instance part="SERIAL" gate="A" x="132.08" y="60.96"/>
-<instance part="C3" gate="G$1" x="114.3" y="81.28" rot="R180"/>
-<instance part="U$8" gate="G$1" x="-30.48" y="299.72"/>
+<instance part="C3" gate="G$1" x="114.3" y="86.36" rot="R180"/>
+<instance part="U$8" gate="G$1" x="-35.56" y="299.72"/>
 <instance part="REG1" gate="A1" x="48.26" y="271.78"/>
 <instance part="D3" gate="1" x="-12.7" y="276.86"/>
@@
 <wire x1="17.78" y1="71.12" x2="20.32" y2="71.12" width="0.1524" layer="91"/>
 <junction x="20.32" y="71.12"/>
+<junction x="27.94" y="68.58"/>
 </segment>
 </net>
@@
 <wire x1="17.78" y1="60.96" x2="20.32" y2="60.96" width="0.1524" layer="91"/>
 <junction x="20.32" y="60.96"/>
+<junction x="27.94" y="63.5"/>
 </segment>
 </net>
@@
 <wire x1="7.62" y1="81.28" x2="7.62" y2="157.48" width="0.1524" layer="91"/>
 <junction x="7.62" y="81.28"/>
+<junction x="27.94" y="81.28"/>
+<junction x="27.94" y="55.88"/>
 </segment>
 <segment>
@@
 <pinref part="OUT_A/MIX" gate="G$1" pin="SLEEVE"/>
 <wire x1="208.28" y1="210.82" x2="210.82" y2="210.82" width="0.1524" layer="91"/>
+<junction x="210.82" y="210.82"/>
+<junction x="187.96" y="190.5"/>
 </segment>
 <segment>
@@
 <junction x="208.28" y="152.4"/>
 <label x="187.96" y="124.46" size="1.778" layer="95"/>
+<junction x="210.82" y="154.94"/>
+<junction x="210.82" y="152.4"/>
+<junction x="210.82" y="149.86"/>
+<junction x="187.96" y="132.08"/>
 </segment>
 <segment>
@@
 <wire x1="96.52" y1="-20.32" x2="99.06" y2="-20.32" width="0.1524" layer="91"/>
 <junction x="96.52" y="-20.32"/>
+<junction x="66.04" y="-20.32"/>
+<junction x="93.98" y="-12.7"/>
 </segment>
 <segment>
@@
 <wire x1="165.1" y1="78.74" x2="167.64" y2="78.74" width="0.1524" layer="91"/>
 <label x="167.64" y="78.74" size="1.778" layer="95"/>
+<junction x="165.1" y="78.74"/>
 </segment>
 <segment>
 <wire x1="165.1" y1="76.2" x2="167.64" y2="76.2" width="0.1524" layer="91"/>
 <label x="167.64" y="76.2" size="1.778" layer="95"/>
+<pinref part="R4" gate="G$1" pin="1"/>
+<junction x="165.1" y="76.2"/>
 </segment>
 </net>
@@
 <junction x="121.92" y="154.94"/>
 <junction x="78.74" y="167.64"/>
+<junction x="27.94" y="78.74"/>
+<junction x="27.94" y="76.2"/>
+<junction x="27.94" y="50.8"/>
+<junction x="116.84" y="185.42"/>
+<junction x="116.84" y="180.34"/>
+<junction x="116.84" y="127"/>
+<junction x="116.84" y="121.92"/>
 </segment>
 <segment>
@@
 <wire x1="81.28" y1="-15.24" x2="81.28" y2="-10.16" width="0.1524" layer="91"/>
 <junction x="81.28" y="-10.16"/>
+<junction x="66.04" y="-10.16"/>
 </segment>
 <segment>
@@
 <junction x="152.4" y="200.66"/>
 <pinref part="C2" gate="G$1" pin="+"/>
+<junction x="116.84" y="200.66"/>
 </segment>
 </net>
@@
 <junction x="157.48" y="142.24"/>
 <pinref part="C1" gate="G$1" pin="+"/>
+<junction x="116.84" y="142.24"/>
 </segment>
 </net>
@@
 <wire x1="142.24" y1="187.96" x2="142.24" y2="213.36" width="0.1524" layer="91"/>
 <label x="142.24" y="213.36" size="1.778" layer="95" rot="R90"/>
+<junction x="116.84" y="187.96"/>
+<junction x="116.84" y="129.54"/>
 </segment>
 <segment>
@@
 <junction x="132.08" y="198.12"/>
 <label x="132.08" y="213.36" size="1.778" layer="95" rot="R90"/>
+<junction x="116.84" y="198.12"/>
+<junction x="116.84" y="139.7"/>
 </segment>
 </net>
@@
 <junction x="134.62" y="195.58"/>
 <label x="134.62" y="213.36" size="1.778" layer="95" rot="R90"/>
+<junction x="116.84" y="195.58"/>
+<junction x="116.84" y="137.16"/>
 </segment>
 </net>
@@
 <junction x="137.16" y="193.04"/>
 <label x="137.16" y="213.36" size="1.778" layer="95" rot="R90"/>
+<junction x="116.84" y="193.04"/>
+<junction x="116.84" y="134.62"/>
 </segment>
 </net>
@@
 <junction x="139.7" y="190.5"/>
 <label x="139.7" y="213.36" size="1.778" layer="95" rot="R90"/>
+<junction x="116.84" y="190.5"/>
+<junction x="116.84" y="132.08"/>
 </segment>
 </net>
@@
 <junction x="124.46" y="203.2"/>
 <label x="124.46" y="213.36" size="1.778" layer="95" rot="R90"/>
+<junction x="116.84" y="203.2"/>
+<junction x="116.84" y="144.78"/>
 </segment>
 </net>
@@
 <junction x="127" y="205.74"/>
 <label x="127" y="213.36" size="1.778" layer="95" rot="R90"/>
+<junction x="116.84" y="205.74"/>
+<junction x="116.84" y="147.32"/>
 </segment>
 </net>
@@
 <junction x="129.54" y="208.28"/>
 <label x="129.54" y="213.36" size="1.778" layer="95" rot="R90"/>
+<junction x="116.84" y="208.28"/>
+<junction x="116.84" y="149.86"/>
 </segment>
 </net>
@@
 <wire x1="116.84" y1="124.46" x2="147.32" y2="124.46" width="0.1524" layer="91"/>
 <label x="144.78" y="124.46" size="1.778" layer="95"/>
+<junction x="116.84" y="124.46"/>
 </segment>
 </net>
@@
 <wire x1="116.84" y1="182.88" x2="147.32" y2="182.88" width="0.1524" layer="91"/>
 <label x="144.78" y="182.88" size="1.778" layer="95"/>
+<junction x="116.84" y="182.88"/>
 </segment>
 </net>
@@
 <pinref part="LEVELA" gate="G$1" pin="W"/>
 <wire x1="177.8" y1="200.66" x2="180.34" y2="200.66" width="0.1524" layer="91"/>
+<junction x="177.8" y="200.66"/>
+<junction x="180.34" y="200.66"/>
 </segment>
 </net>
@@
 <wire x1="190.5" y1="220.98" x2="187.96" y2="220.98" width="0.1524" layer="91"/>
 <wire x1="187.96" y1="220.98" x2="187.96" y2="210.82" width="0.1524" layer="91"/>
+<junction x="187.96" y="210.82"/>
 </segment>
 </net>
@@
 <wire x1="205.74" y1="218.44" x2="205.74" y2="220.98" width="0.1524" layer="91"/>
 <junction x="205.74" y="220.98"/>
+<junction x="210.82" y="220.98"/>
+<junction x="210.82" y="218.44"/>
 </segment>
 </net>
@@
 <wire x1="205.74" y1="157.48" x2="205.74" y2="213.36" width="0.1524" layer="91"/>
 <junction x="205.74" y="213.36"/>
+<junction x="210.82" y="215.9"/>
+<junction x="210.82" y="213.36"/>
+<junction x="210.82" y="157.48"/>
 </segment>
 </net>
@@
 <pinref part="LEVELB" gate="G$1" pin="W"/>
 <wire x1="175.26" y1="142.24" x2="180.34" y2="142.24" width="0.1524" layer="91"/>
+<junction x="175.26" y="142.24"/>
+<junction x="180.34" y="142.24"/>
 </segment>
 </net>
@@
 <pinref part="R8" gate="G$1" pin="2"/>
 <wire x1="187.96" y1="160.02" x2="193.04" y2="160.02" width="0.1524" layer="91"/>
+<junction x="187.96" y="152.4"/>
 </segment>
 </net>
@@
 <pinref part="OUT_B" gate="G$1" pin="TIP"/>
 <wire x1="203.2" y1="160.02" x2="210.82" y2="160.02" width="0.1524" layer="91"/>
+<junction x="210.82" y="160.02"/>
 </segment>
 </net>
@@
 <wire x1="35.56" y1="-12.7" x2="35.56" y2="-10.16" width="0.1524" layer="91"/>
 <junction x="35.56" y="-10.16"/>
+<junction x="40.64" y="-10.16"/>
 </segment>
 </net>
@@
 <wire x1="35.56" y1="-17.78" x2="35.56" y2="-20.32" width="0.1524" layer="91"/>
 <junction x="35.56" y="-20.32"/>
+<junction x="40.64" y="-20.32"/>
 </segment>
 </net>
@@
 <wire x1="68.58" y1="-17.78" x2="111.76" y2="-17.78" width="0.1524" layer="91"/>
 <label x="106.68" y="-17.78" size="1.778" layer="95"/>
+<junction x="66.04" y="-15.24"/>
 </segment>
 <segment>
@@
 <pinref part="R3" gate="G$1" pin="1"/>
 <wire x1="66.04" y1="-12.7" x2="83.82" y2="-12.7" width="0.1524" layer="91"/>
+<junction x="66.04" y="-12.7"/>
+<junction x="83.82" y="-12.7"/>
 </segment>
 </net>
@@
 <wire x1="25.4" y1="93.98" x2="114.3" y2="93.98" width="0.1524" layer="91"/>
 <pinref part="C3" gate="G$1" pin="2"/>
-<wire x1="114.3" y1="93.98" x2="114.3" y2="86.36" width="0.1524" layer="91"/>
+<wire x1="114.3" y1="93.98" x2="114.3" y2="91.44" width="0.1524" layer="91"/>
 <pinref part="R5" gate="G$1" pin="2"/>
 <wire x1="22.86" y1="93.98" x2="25.4" y2="93.98" width="0.1524" layer="91"/>
 <junction x="25.4" y="93.98"/>
+<junction x="114.3" y="91.44"/>
+<junction x="27.94" y="86.36"/>
 </segment>
 </net>
@@
 <wire x1="114.3" y1="68.58" x2="129.54" y2="68.58" width="0.1524" layer="91"/>
 <pinref part="C3" gate="G$1" pin="1"/>
-<wire x1="114.3" y1="78.74" x2="114.3" y2="68.58" width="0.1524" layer="91"/>
+<wire x1="114.3" y1="83.82" x2="114.3" y2="68.58" width="0.1524" layer="91"/>
+<junction x="114.3" y="83.82"/>
 </segment>
 </net>
@@
 <segment>
 <pinref part="U$8" gate="G$1" pin="RING"/>
-<wire x1="-25.4" y1="297.18" x2="-20.32" y2="297.18" width="0.1524" layer="91"/>
+<wire x1="-30.48" y1="297.18" x2="-20.32" y2="297.18" width="0.1524" layer="91"/>
 <wire x1="-20.32" y1="297.18" x2="-20.32" y2="292.1" width="0.1524" layer="91"/>
 <pinref part="U$9" gate="G$1" pin="P$1"/>
@@
 <segment>
 <pinref part="U$8" gate="G$1" pin="TIP"/>
-<wire x1="-25.4" y1="302.26" x2="15.24" y2="302.26" width="0.1524" layer="91"/>
+<wire x1="-30.48" y1="302.26" x2="15.24" y2="302.26" width="0.1524" layer="91"/>
 <wire x1="15.24" y1="302.26" x2="15.24" y2="292.1" width="0.1524" layer="91"/>
 <pinref part="U$9" gate="G$1" pin="P$6"/>
@@
 </segment>
 </net>
-<net name="N$31" class="0">
-<segment>
+<net name="N$20" class="0">
+<segment>
+<pinref part="U$8" gate="G$1" pin="RING_SW"/>
 <pinref part="BATT-" gate="G$1" pin="1"/>
-<pinref part="U$8" gate="G$1" pin="RING_SW"/>
-<wire x1="-25.4" y1="309.88" x2="-25.4" y2="299.72" width="0.1524" layer="91"/>
+<wire x1="-30.48" y1="299.72" x2="-25.4" y2="299.72" width="0.1524" layer="91"/>
+<wire x1="-25.4" y1="299.72" x2="-25.4" y2="309.88" width="0.1524" layer="91"/>
 </segment>
 </net>
@@
 </sheet>
 </sheets>
+<errors>
+</errors>
 </schematic>
 </drawing>

Commit message: more stuff
Parts:
- R6, R7: value (none) -> 470
Connections:
- removed net N$6: OUT_A/MIX.RING, OUT_A/MIX.RING_NC, OUT_B.TIP_NC
- net N$5: now also OUT_B.TIP_NC
Changed lines of the file:
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@@
 <part name="X1" library="crystal" deviceset="CRYSTAL" device="HC49U-V"/>
 <part name="R5" library="rcl" deviceset="R-EU_" device="0207/7"/>
-<part name="R7" library="rcl" deviceset="R-EU_" device="0207/7"/>
+<part name="R7" library="rcl" deviceset="R-EU_" device="0207/7" value="470"/>
 <part name="C4" library="rcl" deviceset="C-EU" device="025-024X044"/>
 <part name="C5" library="rcl" deviceset="C-EU" device="025-024X044"/>
@@
 <part name="C6" library="rcl" deviceset="C-EU" device="025-024X044"/>
 <part name="IC4" library="optocoupler" deviceset="6N138" device=""/>
-<part name="R6" library="rcl" deviceset="R-EU_" device="0207/7"/>
+<part name="R6" library="rcl" deviceset="R-EU_" device="0207/7" value="470"/>
 <part name="LEVELA" library="jasons_stuff" deviceset="ALPS_POT_SMALL" device=""/>
 <part name="C2" library="rcl" deviceset="CPOL-EU" device="E2-5"/>
@@
 <junction x="210.82" y="220.98"/>
 <junction x="210.82" y="218.44"/>
-</segment>
-</net>
-<net name="N$6" class="0">
-<segment>
-<pinref part="OUT_A/MIX" gate="G$1" pin="RING"/>
-<wire x1="210.82" y1="215.9" x2="205.74" y2="215.9" width="0.1524" layer="91"/>
-<wire x1="205.74" y1="215.9" x2="205.74" y2="213.36" width="0.1524" layer="91"/>
-<pinref part="OUT_A/MIX" gate="G$1" pin="RING_NC"/>
-<wire x1="205.74" y1="213.36" x2="210.82" y2="213.36" width="0.1524" layer="91"/>
 <pinref part="OUT_B" gate="G$1" pin="TIP_NC"/>
 <wire x1="210.82" y1="157.48" x2="205.74" y2="157.48" width="0.1524" layer="91"/>
-<wire x1="205.74" y1="157.48" x2="205.74" y2="213.36" width="0.1524" layer="91"/>
-<junction x="205.74" y="213.36"/>
-<junction x="210.82" y="215.9"/>
-<junction x="210.82" y="213.36"/>
+<wire x1="205.74" y1="157.48" x2="205.74" y2="218.44" width="0.1524" layer="91"/>
 <junction x="210.82" y="157.48"/>
-</segment>
-</net>
+<junction x="205.74" y="218.44"/>
+</segment>
+</net>

Commit message: add jumper
Parts:
- added JP3: (no value), pinhead:PINHD-1X3
Connections:
- net CS1: now also JP3.1
- net GND: now also JP3.2
Changed lines of the file:
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@@
 <part name="BATT-" library="pinhead" deviceset="PINHD-1X1" device=""/>
 <part name="BATT+" library="pinhead" deviceset="PINHD-1X1" device=""/>
+<part name="JP3" library="pinhead" deviceset="PINHD-1X3" device=""/>
 </parts>
 <sheets>
@@
 <instance part="BATT-" gate="G$1" x="-25.4" y="312.42" rot="R90"/>
 <instance part="BATT+" gate="G$1" x="-20.32" y="312.42" rot="R90"/>
+<instance part="JP3" gate="A" x="162.56" y="109.22"/>
 </instances>
 <busses>
@@
 <pinref part="R4" gate="G$1" pin="1"/>
 <junction x="165.1" y="76.2"/>
+</segment>
+<segment>
+<pinref part="JP3" gate="A" pin="2"/>
+<wire x1="160.02" y1="109.22" x2="139.7" y2="109.22" width="0.1524" layer="91"/>
+<wire x1="139.7" y1="109.22" x2="139.7" y2="106.68" width="0.1524" layer="91"/>
+<label x="137.16" y="104.14" size="1.778" layer="95"/>
 </segment>
 </net>
@@
 <segment>
 <pinref part="IC3" gate="G$1" pin="CS0#"/>
-<wire x1="116.84" y1="124.46" x2="147.32" y2="124.46" width="0.1524" layer="91"/>
+<wire x1="116.84" y1="124.46" x2="139.7" y2="124.46" width="0.1524" layer="91"/>
 <label x="144.78" y="124.46" size="1.778" layer="95"/>
 <junction x="116.84" y="124.46"/>
-</segment>
-</net>
+<pinref part="JP3" gate="A" pin="1"/>
+<wire x1="139.7" y1="124.46" x2="147.32" y2="124.46" width="0.1524" layer="91"/>
+<wire x1="160.02" y1="111.76" x2="139.7" y2="111.76" width="0.1524" layer="91"/>
+<wire x1="139.7" y1="111.76" x2="139.7" y2="124.46" width="0.1524" layer="91"/>
+<junction x="139.7" y="124.46"/>
+</segment>
+</net>
